Commit message: local change

File: model/urdf/origarmRigidKE.urdf (robot description, URDF)
Before this commit: robot origarmRigidKE, 32 links, 31 joints
Joints:
- joint fixed: origin xyz=0 0 1 rpy=3.141592653589793 0 0 -> xyz=0 0 1 rpy=3.14159265359 0 0
- joint phantom_joint_segment_0_1_beta: limit lower=-6.283185307179586 upper=6.283185307179586 effort=200 velocity=20 -> lower=-6.28318530718 upper=6.28318530718 effort=200 velocity=20
- joint phantom_joint_segment_0_5_betaN: limit lower=-6.283185307179586 upper=6.283185307179586 effort=200 velocity=20 -> lower=-6.28318530718 upper=6.28318530718 effort=200 velocity=20
- joint phantom_joint_segment_1_1_beta: limit lower=-6.283185307179586 upper=6.283185307179586 effort=200 velocity=20 -> lower=-6.28318530718 upper=6.28318530718 effort=200 velocity=20
- joint phantom_joint_segment_1_5_betaN: limit lower=-6.283185307179586 upper=6.283185307179586 effort=200 velocity=20 -> lower=-6.28318530718 upper=6.28318530718 effort=200 velocity=20
- joint phantom_joint_segment_2_1_beta: limit lower=-6.283185307179586 upper=6.283185307179586 effort=200 velocity=20 -> lower=-6.28318530718 upper=6.28318530718 effort=200 velocity=20
- joint phantom_joint_segment_2_5_betaN: limit lower=-6.283185307179586 upper=6.283185307179586 effort=200 velocity=20 -> lower=-6.28318530718 upper=6.28318530718 effort=200 velocity=20
- joint phantom_joint_segment_3_1_beta: limit lower=-6.283185307179586 upper=6.283185307179586 effort=200 velocity=20 -> lower=-6.28318530718 upper=6.28318530718 effort=200 velocity=20
- joint phantom_joint_segment_3_5_betaN: limit lower=-6.283185307179586 upper=6.283185307179586 effort=200 velocity=20 -> lower=-6.28318530718 upper=6.28318530718 effort=200 velocity=20
- joint phantom_joint_segment_4_1_beta: limit lower=-6.283185307179586 upper=6.283185307179586 effort=200 velocity=20 -> lower=-6.28318530718 upper=6.28318530718 effort=200 velocity=20
- joint phantom_joint_segment_4_5_betaN: limit lower=-6.283185307179586 upper=6.283185307179586 effort=200 velocity=20 -> lower=-6.28318530718 upper=6.28318530718 effort=200 velocity=20
- joint phantom_joint_segment_5_1_beta: limit lower=-6.283185307179586 upper=6.283185307179586 effort=200 velocity=20 -> lower=-6.28318530718 upper=6.28318530718 effort=200 velocity=20
- joint phantom_joint_segment_5_5_betaN: limit lower=-6.283185307179586 upper=6.283185307179586 effort=200 velocity=20 -> lower=-6.28318530718 upper=6.28318530718 effort=200 velocity=20
